File: hardware/slave/Slave_Matrix_4x4.kicad_sch (KiCad schematic)
At the start: 48 parts, among them U1 ATtiny1604-SS, U2 74HC153, U3 74AHCT1G125

Commit message: feat(hardware): update Master 4x4 schematic, export PDF, add PCB layout and libraries
Parts:
- C_MOD1, C_MOD10, C_MOD11, C_MOD12, C_MOD13, C_MOD14, C_MOD15, C_MOD16, C_MOD2, C_MOD3, C_MOD4, C_MOD5, C_MOD6, C_MOD7, C_MOD8, C_MOD9: footprint Capacitor_SMD:C_0603_1608Metric -> Capacitor_SMD:C_0805_2012Metric_Pad1.18x1.45mm_HandSolder
Connections:
- net DOUT13: now reaches MOD13.4 (OUT), MOD14.3 (IN)
- net DOUT14: now reaches MOD14.4 (OUT), MOD15.3 (IN)
- net DOUT1: now reaches MOD1.4 (OUT), MOD2.3 (IN)
- net DOUT15: now reaches MOD15.4 (OUT), MOD16.3 (IN)
- net DOUT4: now reaches MOD4.4 (OUT), MOD5.3 (IN)
- net DOUT5: now reaches MOD5.4 (OUT), MOD6.3 (IN)
- net DOUT8: now reaches MOD8.4 (OUT), MOD9.3 (IN)
- net DOUT9: now reaches MOD10.3 (IN), MOD9.4 (OUT)
- net DOUT6: now reaches MOD6.4 (OUT), MOD7.3 (IN)
- net DOUT7: now reaches MOD7.4 (OUT), MOD8.3 (IN)
- net DOUT3: now reaches MOD3.4 (OUT), MOD4.3 (IN)
- net DOUT2: now reaches MOD2.4 (OUT), MOD3.3 (IN)
- net DOUT10: now reaches MOD10.4 (OUT), MOD11.3 (IN)
- net DOUT11: now reaches MOD11.4 (OUT), MOD12.3 (IN)
- net DOUT12: now reaches MOD12.4 (OUT), MOD13.3 (IN)
Changed lines of the file:
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@@
 			)
 		)
-		(property "Footprint" "Capacitor_SMD:C_0603_1608Metric"
+		(property "Footprint" "Capacitor_SMD:C_0805_2012Metric_Pad1.18x1.45mm_HandSolder"
 			(at 191.77 157.48 0)
 			(hide yes)
@@
 			)
 		)
-		(property "Footprint" "Capacitor_SMD:C_0603_1608Metric"
+		(property "Footprint" "Capacitor_SMD:C_0805_2012Metric_Pad1.18x1.45mm_HandSolder"
 			(at 303.53 238.76 0)
 			(hide yes)
@@
 			)
 		)
-		(property "Footprint" "Capacitor_SMD:C_0603_1608Metric"
+		(property "Footprint" "Capacitor_SMD:C_0805_2012Metric_Pad1.18x1.45mm_HandSolder"
 			(at 191.77 116.84 0)
 			(hide yes)
@@
 			)
 		)
-		(property "Footprint" "Capacitor_SMD:C_0603_1608Metric"
+		(property "Footprint" "Capacitor_SMD:C_0805_2012Metric_Pad1.18x1.45mm_HandSolder"
 			(at 359.41 198.12 0)
 			(hide yes)
@@
 			)
 		)
-		(property "Footprint" "Capacitor_SMD:C_0603_1608Metric"
+		(property "Footprint" "Capacitor_SMD:C_0805_2012Metric_Pad1.18x1.45mm_HandSolder"
 			(at 247.65 157.48 0)
 			(hide yes)
@@
 			)
 		)
-		(property "Footprint" "Capacitor_SMD:C_0603_1608Metric"
+		(property "Footprint" "Capacitor_SMD:C_0805_2012Metric_Pad1.18x1.45mm_HandSolder"
 			(at 247.65 198.12 0)
 			(hide yes)
@@
 			)
 		)
-		(property "Footprint" "Capacitor_SMD:C_0603_1608Metric"
+		(property "Footprint" "Capacitor_SMD:C_0805_2012Metric_Pad1.18x1.45mm_HandSolder"
 			(at 247.65 238.76 0)
 			(hide yes)
@@
 			)
 		)
-		(property "Footprint" "Capacitor_SMD:C_0603_1608Metric"
+		(property "Footprint" "Capacitor_SMD:C_0805_2012Metric_Pad1.18x1.45mm_HandSolder"
 			(at 359.41 116.84 0)
 			(hide yes)
@@
 			)
 		)
-		(property "Footprint" "Capacitor_SMD:C_0603_1608Metric"
+		(property "Footprint" "Capacitor_SMD:C_0805_2012Metric_Pad1.18x1.45mm_HandSolder"
 			(at 191.77 198.12 0)
 			(hide yes)
@@
 			)
 		)
-		(property "Footprint" "Capacitor_SMD:C_0603_1608Metric"
+		(property "Footprint" "Capacitor_SMD:C_0805_2012Metric_Pad1.18x1.45mm_HandSolder"
 			(at 359.41 238.76 0)
 			(hide yes)
@@
 			)
 		)
-		(property "Footprint" "Capacitor_SMD:C_0603_1608Metric"
+		(property "Footprint" "Capacitor_SMD:C_0805_2012Metric_Pad1.18x1.45mm_HandSolder"
 			(at 303.53 116.84 0)
 			(hide yes)
@@
 			)
 		)
-		(property "Footprint" "Capacitor_SMD:C_0603_1608Metric"
+		(property "Footprint" "Capacitor_SMD:C_0805_2012Metric_Pad1.18x1.45mm_HandSolder"
 			(at 359.41 157.48 0)
 			(hide yes)
@@
 			)
 		)
-		(property "Footprint" "Capacitor_SMD:C_0603_1608Metric"
+		(property "Footprint" "Capacitor_SMD:C_0805_2012Metric_Pad1.18x1.45mm_HandSolder"
 			(at 303.53 198.12 0)
 			(hide yes)
@@
 			)
 		)
-		(property "Footprint" "Capacitor_SMD:C_0603_1608Metric"
+		(property "Footprint" "Capacitor_SMD:C_0805_2012Metric_Pad1.18x1.45mm_HandSolder"
 			(at 191.77 238.76 0)
 			(hide yes)
@@
 			)
 		)
-		(property "Footprint" "Capacitor_SMD:C_0603_1608Metric"
+		(property "Footprint" "Capacitor_SMD:C_0805_2012Metric_Pad1.18x1.45mm_HandSolder"
 			(at 303.53 157.48 0)
 			(hide yes)
@@
 			)
 		)
-		(property "Footprint" "Capacitor_SMD:C_0603_1608Metric"
+		(property "Footprint" "Capacitor_SMD:C_0805_2012Metric_Pad1.18x1.45mm_HandSolder"
 			(at 247.65 116.84 0)
 			(hide yes)
@@
 	)
 	(embedded_fonts no)
+	(label "DOUT1"
+		(at 205.74 116.84 0)
+		(effects
+			(font
+				(size 1.27 1.27)
+			)
+			(justify left bottom)
+		)
+	)
+	(label "DOUT2"
+		(at 261.62 116.84 0)
+		(effects
+			(font
+				(size 1.27 1.27)
+			)
+			(justify left bottom)
+		)
+	)
+	(label "DOUT3"
+		(at 317.5 116.84 0)
+		(effects
+			(font
+				(size 1.27 1.27)
+			)
+			(justify left bottom)
+		)
+	)
+	(label "DOUT4"
+		(at 264.16 137.16 0)
+		(effects
+			(font
+				(size 1.27 1.27)
+			)
+			(justify left bottom)
+		)
+	)
+	(label "DOUT5"
+		(at 205.74 157.48 0)
+		(effects
+			(font
+				(size 1.27 1.27)
+			)
+			(justify left bottom)
+		)
+	)
+	(label "DOUT6"
+		(at 261.62 157.48 0)
+		(effects
+			(font
+				(size 1.27 1.27)
+			)
+			(justify left bottom)
+		)
+	)
+	(label "DOUT7"
+		(at 317.5 157.48 0)
+		(effects
+			(font
+				(size 1.27 1.27)
+			)
+			(justify left bottom)
+		)
+	)
+	(label "DOUT8"
+		(at 264.16 177.8 0)
+		(effects
+			(font
+				(size 1.27 1.27)
+			)
+			(justify left bottom)
+		)
+	)
+	(label "DOUT9"
+		(at 205.74 198.12 0)
+		(effects
+			(font
+				(size 1.27 1.27)
+			)
+			(justify left bottom)
+		)
+	)
+	(label "DOUT10"
+		(at 261.62 198.12 0)
+		(effects
+			(font
+				(size 1.27 1.27)
+			)
+			(justify left bottom)
+		)
+	)
+	(label "DOUT11"
+		(at 317.5 198.12 0)
+		(effects
+			(font
+				(size 1.27 1.27)
+			)
+			(justify left bottom)
+		)
+	)
+	(label "DOUT12"
+		(at 264.16 218.44 0)
+		(effects
+			(font
+				(size 1.27 1.27)
+			)
+			(justify left bottom)
+		)
+	)
+	(label "DOUT13"
+		(at 205.74 238.76 0)
+		(effects
+			(font
+				(size 1.27 1.27)
+			)
+			(justify left bottom)
+		)
+	)
+	(label "DOUT14"
+		(at 261.62 238.76 0)
+		(effects
+			(font
+				(size 1.27 1.27)
+			)
+			(justify left bottom)
+		)
+	)
+	(label "DOUT15"
+		(at 317.5 238.76 0)
+		(effects
+			(font
+				(size 1.27 1.27)
+			)
+			(justify left bottom)
+		)
+	)
 )

Commit message: feat(hardware): update Master PCB layout and Master/Slave 4x4 matrix schematics
Parts:
- removed J_PWR: DC_5V_IN, TerminalBlock:TerminalBlock_bornier-2_P5.08mm, symbol Connector_Generic:Conn_01x02
- removed MOD1, MOD10, MOD11, MOD12, MOD13, MOD14, MOD15, MOD16, MOD2, MOD3, MOD4, MOD5, MOD6, MOD7, MOD8, MOD9: WCMCU-2812-4, Module:CJMCU-2812-4, symbol Custom:CJMCU-2812-4
- added D_TVS1: SMAJ5.0A, Diode_SMD:D_SMA, symbol Device:D_TVS
- added MOD1, MOD10, MOD11, MOD12, MOD13, MOD14, MOD15, MOD16, MOD2, MOD3, MOD4, MOD5, MOD6, MOD7, MOD8, MOD9: WS2812_Matrix_2x2, ws2812-matrix-2x2:WS2812_Matrix_2x2_15x15mm, symbol ws2812-matrix-2x2:WS2812_Matrix_2x2
- C2: value 10u -> 100uF; footprint Capacitor_SMD:C_0805_2012Metric -> Capacitor_SMD:C_1206_3216Metric
- C_MOD1, C_MOD10, C_MOD11, C_MOD12, C_MOD13, C_MOD14, C_MOD15, C_MOD16, C_MOD2, C_MOD3, C_MOD4, C_MOD5, C_MOD6, C_MOD7, C_MOD8, C_MOD9: footprint Capacitor_SMD:C_0805_2012Metric_Pad1.18x1.45mm_HandSolder -> Capacitor_SMD:C_0805_2012Metric
Connections:
- net +5V: now also D_TVS1.1 (A1), MOD1.2 (VCC_IN), MOD1.6 (VCC_OUT), MOD10.2 (VCC_IN), MOD10.6 (VCC_OUT), MOD11.2 (VCC_IN), MOD11.6 (VCC_OUT), MOD12.2 (VCC_IN), MOD12.6 (VCC_OUT), MOD13.2 (VCC_IN), MOD13.6 (VCC_OUT), MOD14.2 (VCC_IN), MOD14.6 (VCC_OUT), MOD15.2 (VCC_IN), MOD15.6 (VCC_OUT), MOD16.2 (VCC_IN), MOD16.6 (VCC_OUT), MOD2.2 (VCC_IN), MOD2.6 (VCC_OUT), MOD3.2 (VCC_IN), MOD3.6 (VCC_OUT), MOD4.2 (VCC_IN), MOD4.6 (VCC_OUT), MOD5.2 (VCC_IN), MOD5.6 (VCC_OUT), MOD6.2 (VCC_IN), MOD6.6 (VCC_OUT), MOD7.2 (VCC_IN), MOD7.6 (VCC_OUT), MOD8.2 (VCC_IN), MOD8.6 (VCC_OUT), MOD9.2 (VCC_IN), MOD9.6 (VCC_OUT)
- net DIN_LOCAL: now also MOD1.3 (DIN)
- net DOUT12: now also MOD12.7 (DOUT), MOD13.3 (DIN)
- net DOUT4: now also MOD4.7 (DOUT), MOD5.3 (DIN)
- net DOUT8: now also MOD8.7 (DOUT), MOD9.3 (DIN)
- net DOUT_LOCAL: now also MOD16.7 (DOUT)
- net GND: now also D_TVS1.2 (A2), MOD1.1 (GND_IN1), MOD1.4 (GND_IN2), MOD1.5 (GND_OUT1), MOD1.8 (GND_OUT2), MOD10.1 (GND_IN1), MOD10.4 (GND_IN2), MOD10.5 (GND_OUT1), MOD10.8 (GND_OUT2), MOD11.1 (GND_IN1), MOD11.4 (GND_IN2), MOD11.5 (GND_OUT1), MOD11.8 (GND_OUT2), MOD12.1 (GND_IN1), MOD12.4 (GND_IN2), MOD12.5 (GND_OUT1), MOD12.8 (GND_OUT2), MOD13.1 (GND_IN1), MOD13.4 (GND_IN2), MOD13.5 (GND_OUT1), MOD13.8 (GND_OUT2), MOD14.1 (GND_IN1), MOD14.4 (GND_IN2), MOD14.5 (GND_OUT1), MOD14.8 (GND_OUT2), MOD15.1 (GND_IN1), MOD15.4 (GND_IN2), MOD15.5 (GND_OUT1), MOD15.8 (GND_OUT2), MOD16.1 (GND_IN1), MOD16.4 (GND_IN2), MOD16.5 (GND_OUT1), MOD16.8 (GND_OUT2), MOD2.1 (GND_IN1), MOD2.4 (GND_IN2), MOD2.5 (GND_OUT1), MOD2.8 (GND_OUT2), MOD3.1 (GND_IN1), MOD3.4 (GND_IN2), MOD3.5 (GND_OUT1), MOD3.8 (GND_OUT2), MOD4.1 (GND_IN1), MOD4.4 (GND_IN2), MOD4.5 (GND_OUT1), MOD4.8 (GND_OUT2), MOD5.1 (GND_IN1), MOD5.4 (GND_IN2), MOD5.5 (GND_OUT1), MOD5.8 (GND_OUT2), MOD6.1 (GND_IN1), MOD6.4 (GND_IN2), MOD6.5 (GND_OUT1), MOD6.8 (GND_OUT2), MOD7.1 (GND_IN1), MOD7.4 (GND_IN2), MOD7.5 (GND_OUT1), MOD7.8 (GND_OUT2), MOD8.1 (GND_IN1), MOD8.4 (GND_IN2), MOD8.5 (GND_OUT1), MOD8.8 (GND_OUT2), MOD9.1 (GND_IN1), MOD9.4 (GND_IN2), MOD9.5 (GND_OUT1), MOD9.8 (GND_OUT2)
- new net: MOD10.7 (DOUT), MOD11.3 (DIN)
- new net: MOD11.7 (DOUT), MOD12.3 (DIN)
- new net: MOD5.7 (DOUT), MOD6.3 (DIN)
- new net: MOD6.7 (DOUT), MOD7.3 (DIN)
- new net: MOD14.7 (DOUT), MOD15.3 (DIN)
- new net: MOD15.7 (DOUT), MOD16.3 (DIN)
- new net: MOD1.7 (DOUT), MOD2.3 (DIN)
- new net: MOD13.7 (DOUT), MOD14.3 (DIN)
- new net: MOD10.3 (DIN), MOD9.7 (DOUT)
- new net: MOD3.7 (DOUT), MOD4.3 (DIN)
- new net: MOD2.7 (DOUT), MOD3.3 (DIN)
- new net: MOD7.7 (DOUT), MOD8.3 (DIN)
Other:
- note added: "1. ATTINY1604 NEIGHBOR SENSE & MUX LOGIC"
- note added: "2. 74HC153 4-TO-1 MUX & 74AHCT1G125 BUFFER"
- note added: "3. MAGNETIC EDGE CONNECTORS (SYMMETRICAL MATING & DOUT STREAM)"
- note added: "3. POWER INPUT & SURGE PROTECTION (TVS & BULK CAP)"
- note added: "SLAVE EXPANSION BOARD - AUTONOMOUS 4-WAY AUTO-ROUTING MATRIX"
- note removed: "1. SLAVE CONTROLLER (ATtiny1604-SS) & UPDI INTERFACE"
- note removed: "2. AUTO-ROUTING MULTIPLEXER & DRIVER (74HC153 + 74AHCT1G125)"
- note removed: "3. POWER DISTRIBUTION & DC INPUT"
- note removed: "4. MAGNETIC EDGE CONNECTORS (SYMMETRICAL MATING & PASS-THROUGH)"
- note removed: "5. SMART LED MATRIX 4x4 (LEFT-TO-RIGHT CLEAN FLOW -> DOUT_LOCAL)"
- moved on the sheet: C1, C2, C3, C4, D1, J_PROG, R_LED, R_UPDI, U2, U3

Commit message: feat(hardware): update schematics, symbol libraries, and system architecture docs
- Update Master and Slave 4x4 matrix schematics with proper data flow pipeline and symbol pinouts
- Align symbol libraries (esp32-wemos-d1-mini, ws2812-matrix-2x2) across common and local folders
- Update project README and hardware documentation for VBUS power distribution, level shifting, and data flow architecture
Parts:
- removed C4: 100n, Capacitor_SMD:C_0603_1608Metric, symbol Device:C
- removed U2: 74HC153, Package_SO:SOIC-16_3.9x9.9mm_P1.27mm, symbol 74xx:74HC153
- added R_BUS: DNP, Resistor_SMD:R_2512_6332Metric, symbol Device:R
- D_TVS1: value SMAJ5.0A -> D_TVS
Connections:
- net DATA_N is gone; now on net LINK_TX: J_NORTH.3
- net DATA_S is gone; now on net LINK_TX: J_SOUTH.2
- net DATA_W is gone; now on net LINK_TX: J_WEST.2
- net MUX_EN is gone; now on net LINK_TX: U1.7 (PB2)
- net MUX_S0 is gone; now on net LED_DATA: U1.9 (PB0)
- net MUX_S1 is gone; now on net LED_STATUS: U1.8 (PB1)
- net +5V: now also R_BUS.2; no longer D_TVS1.1 (A1), J_EAST.4, J_NORTH.4, J_SOUTH.1, J_WEST.1
- net GND: now also J_SOUTH.1, J_WEST.1; no longer J_SOUTH.4, J_WEST.4
- net LED_STATUS: no longer U1.6 (PB3)
- net LED_DATA: now reaches U3.2 (A)
- net DATA_E renamed LINK_TX
- net DOUT_LOCAL: no longer names the net of MOD16.7 (DOUT)
- net SENSE_E renamed LINK_RX_E
- net SENSE_N renamed LINK_RX_N
- net SENSE_S renamed LINK_RX_S
- net SENSE_W renamed LINK_RX_W
- new net VBUS: D_TVS1.1 (A1), J_EAST.4, J_NORTH.4, J_SOUTH.4, J_WEST.4, R_BUS.1
- no-connect marks 4 -> 5
Other:
- note added: "1. ATTINY1604 NEIGHBOR RX & ROUTING LOGIC"
- note added: "2. LOCAL LED OUTPUT BUFFER (74AHCT1G125)"
- note added: "3. MAGNETIC EDGE CONNECTORS (SYMMETRICAL LINK BUS)"
- note added: "4. POWER INPUT & SURGE PROTECTION (TVS & BULK CAP)"
- note removed: "1. ATTINY1604 NEIGHBOR SENSE & MUX LOGIC"
- note removed: "2. 74HC153 4-TO-1 MUX & 74AHCT1G125 BUFFER"
- note removed: "3. MAGNETIC EDGE CONNECTORS (SYMMETRICAL MATING & DOUT STREAM)"
- note removed: "3. POWER INPUT & SURGE PROTECTION (TVS & BULK CAP)"
